Commit message: checkpoint(05-08): align dummy feedback and desktop diagnostics

File: shared/robot-profiles/BuiltIn/dummy-6dof/model/dummy.urdf (robot description, URDF)
Before this commit: robot dummy, 7 links, 6 joints
Joints:
- joint joint_1: limit lower=-3.14 upper=3.14 effort=0 velocity=0 -> lower=-2.9670597284 upper=2.9670597284 effort=0 velocity=0
- joint joint_2: limit lower=-1.30 upper=2.18 effort=0 velocity=0 -> lower=-1.3089969390 upper=1.5707963268 effort=0 velocity=0
- joint joint_3: limit lower=-1.63 upper=1.60 effort=0 velocity=0 -> lower=-1.5707963268 upper=1.5707963268 effort=0 velocity=0
- joint joint_4: limit lower=-3.14 upper=3.14 effort=0 velocity=0 -> lower=-3.1415926536 upper=3.1415926536 effort=0 velocity=0
- joint joint_5: limit lower=-1.76 upper=1.76 effort=0 velocity=0 -> lower=-2.0943951024 upper=2.0943951024 effort=0 velocity=0
- joint joint_6: limit lower=-3.14 upper=3.14 effort=0 velocity=0 -> lower=-12.5663706144 upper=12.5663706144 effort=0 velocity=0
