Commit message: phase(A0-R1): replace Aethor deployed model

File: shared/robot-profiles/BuiltIn/aethor-robo-dual-7dof/model/aethor_robo.urdf (robot description, URDF)
Before this commit: robot aethor_robo, 23 links, 22 joints
Links:
- removed link wheel_link_1
- removed link wheel_link_2
- removed link wheel_link_3
- removed link wheel_link_4
- removed link wheel_link_5
- removed link wheel_link_6
- link left_arm_base_link: mass 0.279378451395946 -> 0.279378451396139
- link left_arm_link_1: mass 0.365875053527118 -> 0.365875053527311
- link left_arm_link_2: mass 0.456775467385593 -> 0.456775467385786
- link left_arm_link_3: mass 0.510338228721455 -> 0.510338228721648
- link left_arm_link_4: mass 0.456903524845923 -> 0.456903524846116
- link left_arm_link_5: mass 0.289103221587114 -> 0.289103221587113
- link left_arm_link_6: mass 0.660923355971569 -> 0.660923355971955
- link left_arm_link_7: mass 0.889614130479029 -> 0.88961412966904
- link right_arm_base_link: mass 0.279378451116301 -> 0.279378451116494
- link right_arm_link_1: mass 0.365875053503755 -> 0.365875053503948
- link right_arm_link_2: mass 0.456775477069743 -> 0.456775477069936
- link right_arm_link_3: mass 0.510338228879153 -> 0.510338228879347
- link right_arm_link_4: mass 0.45690352484592 -> 0.456903524846113
- link right_arm_link_6: mass 0.660923355736345 -> 0.660923355736731
- link right_arm_link_7: mass 0.889614117986897 -> 0.889614113446627
- link satellite_base_link: mass 94.6839838101448 -> 94.6839838100833
Joints:
- removed joint wheel_joint_1
- removed joint wheel_joint_2
- removed joint wheel_joint_3
- removed joint wheel_joint_4
- removed joint wheel_joint_5
- removed joint wheel_joint_6
- joint left_arm_joint_2: origin xyz=0 0.0384 0.0722 rpy=1.5708 -1.5708 0 -> xyz=0 0.0384 0.0722 rpy=1.5707963267949 -1.5707963267949 0
- joint left_arm_joint_3: origin xyz=0 0.30833 0.028 rpy=1.5708 0 3.1416 -> xyz=0 0.308325 0.0279999999999999 rpy=1.5707963267949 0 3.14159265358979
- joint left_arm_joint_4: origin xyz=0 0.0387 0.4322 rpy=-1.5708 0 0 -> xyz=0 0.0387 0.4322 rpy=-1.5707963267949 0 0
- joint left_arm_joint_5: origin xyz=0 0.30833 0.028 rpy=1.5708 0 3.1416 -> xyz=0 0.308325 0.0279999999999999 rpy=1.5707963267949 0 3.14159265358979
- joint left_arm_joint_6: origin xyz=0 0.028 0.482 rpy=1.5708 0 0 -> xyz=0 0.0280000000000005 0.482 rpy=1.5707963267949 0 0
- joint left_arm_joint_7: origin xyz=0 -0.21653 -0.0387 rpy=-1.5708 0 3.1416 -> xyz=0 -0.216525 -0.0387000000000002 rpy=-1.5707963267949 0 3.14159265358979
- joint left_arm_mount_joint: origin xyz=0.431 0.199 -0.071218 rpy=1.5708 0 3.1416 -> xyz=0.431000000000001 0.199 -0.0712182540694777 rpy=1.5707963267949 0 3.14159265358979
- joint right_arm_joint_2: origin xyz=0 0.038 0.0722 rpy=1.5708 -1.5708 0 -> xyz=0 0.038 0.0722 rpy=1.5707963267949 -1.5707963267949 0
- joint right_arm_joint_3: origin xyz=0 -0.30833 0.0284 rpy=1.5708 0 0 -> xyz=0 -0.308325 0.0284000000000002 rpy=1.5707963267949 0 0
- joint right_arm_joint_4: origin xyz=0 0.038 0.4322 rpy=-1.5708 0 0 -> xyz=0 0.0380000000000003 0.4322 rpy=-1.5707963267949 0 0
- joint right_arm_joint_5: origin xyz=0 0.30833 0.0287 rpy=1.5708 0 3.1416 -> xyz=0 0.308325 0.0286999999999997 rpy=1.5707963267949 0 3.14159265358979
- joint right_arm_joint_6: origin xyz=0 0.028 0.482 rpy=1.5708 0 0 -> xyz=0 0.0279999999999996 0.482 rpy=1.5707963267949 0 0
- joint right_arm_joint_7: origin xyz=0 -0.21653 -0.0387 rpy=-1.5708 0 3.1416 -> xyz=0 -0.216525 -0.0387000000000006 rpy=-1.5707963267949 0 3.14159265358979
- joint right_arm_mount_joint: origin xyz=0.431 -0.199 -0.071218 rpy=1.5708 0 0 -> xyz=0.431000000000001 -0.199 -0.0712182540694777 rpy=1.5707963267949 0 0
